Commit message: URDF

File: src/biped_description/urdf/biped.urdf.xacro (robot description, xacro)
@@ -1,4 +1,48 @@
 <?xml version="1.0"?>
 <robot xmlns:xacro="http://www.ros.org/wiki/xacro" name="biped">
+  <!-- ros2_control hardware interface configuration -->
+  <ros2_control name="BipedSystem" type="system">
+    <hardware>
+      <plugin>gazebo_ros2_control/GazeboSystem</plugin>
+    </hardware>
+    <joint name="left_hip_roll_joint">
+      <command_interface name="position"/>
+      <state_interface name="position"/>
+      <state_interface name="velocity"/>
+    </joint>
+    <joint name="left_knee_joint">
+      <command_interface name="position"/>
+      <state_interface name="position"/>
+      <state_interface name="velocity"/>
+    </joint>
+    <joint name="left_ankle_joint">
+      <command_interface name="position"/>
+      <state_interface name="position"/>
+      <state_interface name="velocity"/>
+    </joint>
+    <joint name="right_hip_roll_joint">
+      <command_interface name="position"/>
+      <state_interface name="position"/>
+      <state_interface name="velocity"/>
+    </joint>
+    <joint name="right_knee_joint">
+      <command_interface name="position"/>
+      <state_interface name="position"/>
+      <state_interface name="velocity"/>
+    </joint>
+    <joint name="right_ankle_joint">
+      <command_interface name="position"/>
+      <state_interface name="position"/>
+      <state_interface name="velocity"/>
+    </joint>
+  </ros2_control>
+  <gazebo>
+    <plugin name="gazebo_ros2_control" filename="libgazebo_ros2_control.so">
+      <ros2_control>
+        <param name="update_rate">100</param>
+        <param name="config_file">/home/yogesh_rajesh/biped_ros2_ws/src/biped_description/config/biped_controllers.yaml</param>
+      </ros2_control>
+    </plugin>
+  </gazebo>
   <!-- Torso Link -->
   <link name="torso_link">
@@ -31,12 +75,4 @@
       </imu>
     </sensor>
-  </gazebo>
-  <gazebo>
-    <plugin name="gazebo_ros2_control" filename="libgazebo_ros2_control.so">
-      <ros2_control>
-        <param name="update_rate">100</param>
-        <param name="config_file">/home/yogesh_rajesh/biped_ros2_ws/src/biped_description/config/biped_controllers.yaml</param>
-      </ros2_control>
-    </plugin>
   </gazebo>
   <!-- Left Hip Joint -->

Commit message: MPC control

File: src/biped_description/urdf/biped.urdf.xacro (robot description, xacro)
@@ -1,48 +1,4 @@
 <?xml version="1.0"?>
 <robot xmlns:xacro="http://www.ros.org/wiki/xacro" name="biped">
-  <!-- ros2_control hardware interface configuration -->
-  <ros2_control name="BipedSystem" type="system">
-    <hardware>
-      <plugin>gazebo_ros2_control/GazeboSystem</plugin>
-    </hardware>
-    <joint name="left_hip_roll_joint">
-      <command_interface name="position"/>
-      <state_interface name="position"/>
-      <state_interface name="velocity"/>
-    </joint>
-    <joint name="left_knee_joint">
-      <command_interface name="position"/>
-      <state_interface name="position"/>
-      <state_interface name="velocity"/>
-    </joint>
-    <joint name="left_ankle_joint">
-      <command_interface name="position"/>
-      <state_interface name="position"/>
-      <state_interface name="velocity"/>
-    </joint>
-    <joint name="right_hip_roll_joint">
-      <command_interface name="position"/>
-      <state_interface name="position"/>
-      <state_interface name="velocity"/>
-    </joint>
-    <joint name="right_knee_joint">
-      <command_interface name="position"/>
-      <state_interface name="position"/>
-      <state_interface name="velocity"/>
-    </joint>
-    <joint name="right_ankle_joint">
-      <command_interface name="position"/>
-      <state_interface name="position"/>
-      <state_interface name="velocity"/>
-    </joint>
-  </ros2_control>
-  <gazebo>
-    <plugin name="gazebo_ros2_control" filename="libgazebo_ros2_control.so">
-      <ros2_control>
-        <param name="update_rate">100</param>
-        <param name="config_file">/home/yogesh_rajesh/biped_ros2_ws/src/biped_description/config/biped_controllers.yaml</param>
-      </ros2_control>
-    </plugin>
-  </gazebo>
   <!-- Torso Link -->
   <link name="torso_link">
@@ -61,7 +17,7 @@
     </collision>
     <inertial>
-      <mass value="5.0"/>
-      <origin xyz="0 0 0" rpy="0 0 0"/>
-      <inertia ixx="0.054" iyy="0.083" izz="0.021" ixy="0.0" ixz="0.0" iyz="0.0"/>
+      <mass value="34.9"/>
+      <origin xyz="0 0 0" rpy="0 0 0"/>
+      <inertia ixx="0.327" iyy="0.131" izz="0.327" ixy="0.0" ixz="0.0" iyz="0.0"/>
     </inertial>
   </link>
@@ -88,8 +44,8 @@
     <type>transmission_interface/SimpleTransmission</type>
     <joint name="left_hip_roll_joint">
-      <hardwareInterface>PositionJointInterface</hardwareInterface>
+      <hardwareInterface>position</hardwareInterface>
     </joint>
     <actuator name="left_hip_motor">
-      <hardwareInterface>PositionJointInterface</hardwareInterface>
+      <hardwareInterface>position</hardwareInterface>
       <mechanicalReduction>1</mechanicalReduction>
     </actuator>
@@ -113,7 +69,7 @@
     </collision>
     <inertial>
-      <mass value="0.8"/>
-      <origin xyz="0 0 -0.11" rpy="0 0 0"/>
-      <inertia ixx="0.00299" iyy="0.00299" izz="0.00064" ixy="0.0" ixz="0.0" iyz="0.0"/>
+      <mass value="5.58"/>
+      <origin xyz="0 0 -0.11" rpy="0 0 0"/>
+      <inertia ixx="0.0242" iyy="0.0242" izz="0.00342" ixy="0.0" ixz="0.0" iyz="0.0"/>
     </inertial>
   </link>
@@ -130,8 +86,8 @@
     <type>transmission_interface/SimpleTransmission</type>
     <joint name="left_knee_joint">
-      <hardwareInterface>PositionJointInterface</hardwareInterface>
+      <hardwareInterface>position</hardwareInterface>
     </joint>
     <actuator name="left_knee_motor">
-      <hardwareInterface>PositionJointInterface</hardwareInterface>
+      <hardwareInterface>position</hardwareInterface>
       <mechanicalReduction>1</mechanicalReduction>
     </actuator>
@@ -155,7 +111,7 @@
     </collision>
     <inertial>
-      <mass value="0.6"/>
-      <origin xyz="0 0 -0.1" rpy="0 0 0"/>
-      <inertia ixx="0.00224" iyy="0.00224" izz="0.00048" ixy="0.0" ixz="0.0" iyz="0.0"/>
+      <mass value="4.19"/>
+      <origin xyz="0 0 -0.1" rpy="0 0 0"/>
+      <inertia ixx="0.0280" iyy="0.0280" izz="0.00131" ixy="0.0" ixz="0.0" iyz="0.0"/>
     </inertial>
   </link>
@@ -172,8 +128,8 @@
     <type>transmission_interface/SimpleTransmission</type>
     <joint name="left_ankle_joint">
-      <hardwareInterface>PositionJointInterface</hardwareInterface>
+      <hardwareInterface>position</hardwareInterface>
     </joint>
     <actuator name="left_ankle_motor">
-      <hardwareInterface>PositionJointInterface</hardwareInterface>
+      <hardwareInterface>position</hardwareInterface>
       <mechanicalReduction>1</mechanicalReduction>
     </actuator>
@@ -207,7 +163,7 @@
     </collision>
     <inertial>
-      <mass value="0.4"/>
-      <origin xyz="0 0 0" rpy="0 0 0"/>
-      <inertia ixx="0.0004" iyy="0.0004" izz="0.0004" ixy="0.0" ixz="0.0" iyz="0.0"/>
+      <mass value="2.79"/>
+      <origin xyz="0 0 0" rpy="0 0 0"/>
+      <inertia ixx="0.00279" iyy="0.00279" izz="0.00279" ixy="0.0" ixz="0.0" iyz="0.0"/>
     </inertial>
   </link>
@@ -224,8 +180,8 @@
     <type>transmission_interface/SimpleTransmission</type>
     <joint name="right_hip_roll_joint">
-      <hardwareInterface>PositionJointInterface</hardwareInterface>
+      <hardwareInterface>position</hardwareInterface>
     </joint>
     <actuator name="right_hip_motor">
-      <hardwareInterface>PositionJointInterface</hardwareInterface>
+      <hardwareInterface>position</hardwareInterface>
       <mechanicalReduction>1</mechanicalReduction>
     </actuator>
@@ -249,7 +205,7 @@
     </collision>
     <inertial>
-      <mass value="0.8"/>
-      <origin xyz="0 0 -0.11" rpy="0 0 0"/>
-      <inertia ixx="0.00299" iyy="0.00299" izz="0.00064" ixy="0.0" ixz="0.0" iyz="0.0"/>
+      <mass value="5.58"/>
+      <origin xyz="0 0 -0.11" rpy="0 0 0"/>
+      <inertia ixx="0.0236" iyy="0.0236" izz="0.0034" ixy="0.0" ixz="0.0" iyz="0.0"/>
     </inertial>
   </link>
@@ -266,8 +222,8 @@
     <type>transmission_interface/SimpleTransmission</type>
     <joint name="right_knee_joint">
-      <hardwareInterface>PositionJointInterface</hardwareInterface>
+      <hardwareInterface>position</hardwareInterface>
     </joint>
     <actuator name="right_knee_motor">
-      <hardwareInterface>PositionJointInterface</hardwareInterface>
+      <hardwareInterface>position</hardwareInterface>
       <mechanicalReduction>1</mechanicalReduction>
     </actuator>
@@ -291,7 +247,7 @@
     </collision>
     <inertial>
-      <mass value="0.6"/>
-      <origin xyz="0 0 -0.1" rpy="0 0 0"/>
-      <inertia ixx="0.00224" iyy="0.00224" izz="0.00048" ixy="0.0" ixz="0.0" iyz="0.0"/>
+      <mass value="4.19"/>
+      <origin xyz="0 0 -0.1" rpy="0 0 0"/>
+      <inertia ixx="0.0280" iyy="0.0280" izz="0.00066" ixy="0.0" ixz="0.0" iyz="0.0"/>
     </inertial>
   </link>
@@ -308,8 +264,8 @@
     <type>transmission_interface/SimpleTransmission</type>
     <joint name="right_ankle_joint">
-      <hardwareInterface>PositionJointInterface</hardwareInterface>
+      <hardwareInterface>position</hardwareInterface>
     </joint>
     <actuator name="right_ankle_motor">
-      <hardwareInterface>PositionJointInterface</hardwareInterface>
+      <hardwareInterface>position</hardwareInterface>
       <mechanicalReduction>1</mechanicalReduction>
     </actuator>
@@ -343,8 +299,50 @@
     </collision>
     <inertial>
-      <mass value="0.4"/>
-      <origin xyz="0 0 0" rpy="0 0 0"/>
-      <inertia ixx="0.0004" iyy="0.0004" izz="0.0004" ixy="0.0" ixz="0.0" iyz="0.0"/>
-    </inertial>
-  </link>
+      <mass value="2.79"/>
+      <origin xyz="0 0 0" rpy="0 0 0"/>
+      <inertia ixx="0.00279" iyy="0.00279" izz="0.00279" ixy="0.0" ixz="0.0" iyz="0.0"/>
+    </inertial>
+  </link>
+  <!-- ros2_control hardware interface configuration -->
+  <ros2_control name="BipedSystem" type="system">
+    <hardware>
+      <plugin>gazebo_ros2_control/GazeboSystem</plugin>
+    </hardware>
+    <joint name="left_hip_roll_joint">
+      <command_interface name="position"/>
+      <state_interface name="position"/>
+      <state_interface name="velocity"/>
+    </joint>
+    <joint name="left_knee_joint">
+      <command_interface name="position"/>
+      <state_interface name="position"/>
+      <state_interface name="velocity"/>
+    </joint>
+    <joint name="left_ankle_joint">
+      <command_interface name="position"/>
+      <state_interface name="position"/>
+      <state_interface name="velocity"/>
+    </joint>
+    <joint name="right_hip_roll_joint">
+      <command_interface name="position"/>
+      <state_interface name="position"/>
+      <state_interface name="velocity"/>
+    </joint>
+    <joint name="right_knee_joint">
+      <command_interface name="position"/>
+      <state_interface name="position"/>
+      <state_interface name="velocity"/>
+    </joint>
+    <joint name="right_ankle_joint">
+      <command_interface name="position"/>
+      <state_interface name="position"/>
+      <state_interface name="velocity"/>
+    </joint>
+  </ros2_control>
+  <gazebo>
+    <plugin name="gazebo_ros2_control" filename="libgazebo_ros2_control.so">
+      <robot_namespace>/</robot_namespace>
+      <parameters>/home/yogesh_rajesh/biped_ros2_ws/src/biped_description/config/biped_controllers.yaml</parameters>
+    </plugin>
+  </gazebo>
 </robot>
